File: hardware/pcb/audio_player_toy_v1/audio_player_toy_v1.kicad_sch (KiCad schematic)
At the start: 13 parts, among them J1 Conn_02x05_Odd_Even, U1 BH-AAA-B5AA005, U2 ISD2360YYI

Commit message: doc: generate BOM for v1 and v2
Parts:
- R1: Component (none) -> RC0603FR-0710KL; Detail (none) -> +-1%, 100mW; Manufactor (none) -> Yageo
Changed lines of the file:
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@@
 			)
 		)
-		(property "Manufactor" ""
+		(property "Manufactor" "Yageo"
 			(at 63.5 55.88 0)
 			(effects
+				(font
+					(size 1.27 1.27)
+				)
+				(hide yes)
+			)
+		)
+		(property "Component" "RC0603FR-0710KL"
+			(at 63.5 55.88 0)
+			(effects
+				(font
+					(size 1.27 1.27)
+				)
+				(hide yes)
+			)
+		)
+		(property "Detail" "+-1%, 100mW"
+			(at 63.5 55.88 0)
+			(effects
